File: Hardware/Wake-up Light Controller.brd (EAGLE design)
At the start: 85.7 x 54 mm, 48 parts, among them IC1 ST1S10, IC2 HT7333, IC3 DS3231/SO, IC4 ATMEGA328P_TQFP, J1 AVR-ISP, J2 Debug, J3 CR1632_3V, Q1 BSS138, Q2 BSS138, Q3 FDN306P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

Commit message: Changed component value
Add "debug" value to jumper JP1
Parts:
- JP1: value (none) -> Debug
Changed lines of the file:
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@@
 <layer number="37" name="tTest" color="7" fill="1" visible="no" active="yes"/>
 <layer number="38" name="bTest" color="7" fill="1" visible="no" active="yes"/>
-<layer number="39" name="tKeepout" color="4" fill="11" visible="no" active="yes"/>
-<layer number="40" name="bKeepout" color="1" fill="11" visible="no" active="yes"/>
+<layer number="39" name="tKeepout" color="4" fill="11" visible="yes" active="yes"/>
+<layer number="40" name="bKeepout" color="1" fill="11" visible="yes" active="yes"/>
 <layer number="41" name="tRestrict" color="4" fill="10" visible="yes" active="yes"/>
 <layer number="42" name="bRestrict" color="1" fill="10" visible="yes" active="yes"/>
@@
 <attribute name="VALUE" x="25.55875" y="25.4" size="1" layer="27" rot="R180"/>
 </element>
-<element name="JP1" library="jumper" library_urn="urn:adsk.eagle:library:252" package="JP2" package3d_urn="urn:adsk.eagle:package:15452/1" value="" x="8.255" y="46.355" smashed="yes" rot="R180">
+<element name="JP1" library="jumper" library_urn="urn:adsk.eagle:library:252" package="JP2" package3d_urn="urn:adsk.eagle:package:15452/1" value="Debug" x="8.255" y="46.355" smashed="yes" rot="R180">
 <attribute name="NAME" x="6.4135" y="44.704" size="1" layer="25" ratio="10" rot="R180"/>
 <attribute name="VALUE" x="11.811" y="50.673" size="1.27" layer="27" ratio="10" rot="R180"/>
